File: _autosave-BaseAurora.kicad_pcb (KiCad board)
At the start: 2 copper layers, 80 x 100 mm, 43 parts, among them J1 Conn_01x04_Male, J10 Conn_01x03_Male, J11 Screw_Terminal_01x02, J2 Conn_01x05_Male, J3 Screw_Terminal_01x02, J4 Conn_01x04_Male, J5 Conn_01x04_Male, J6 Screw_Terminal_01x02, J7 Screw_Terminal_01x02, J8 Header_1x2, J9 Header_1x2, K1 HK4100F-DC3V-SHG, Q1 2N3906, Q2 PN2222A, U1 ME6217C33M5G, U2 E32-915T20D, U3 4N32M, U4 NodeMCU1.0(ESP-12E)

Commit message: Design inicial da pcb
Changed lines of the file:
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@@
   )
   (setup
-    (last_trace_width 0.3)
+    (last_trace_width 2)
     (user_trace_width 0.2)
     (user_trace_width 0.3)
@@
   (segment (start 218.7 32.70002) (end 218.37499 32.37501) (width 0.3) (layer F.Cu) (net 1))
   (segment (start 218.37499 32.37501) (end 218.110008 32.37501) (width 0.6) (layer F.Cu) (net 1))
-  (segment (start 218.7 35.25) (end 218.7 32.70002) (width 0.6) (layer F.Cu) (net 1))
+  (segment (start 218.7 35.25) (end 218.7 32.70002) (width 0.3) (layer F.Cu) (net 1))
   (segment (start 225.239956 32.37501) (end 218.37499 32.37501) (width 0.6) (layer F.Cu) (net 1))
   (segment (start 222.45625 27.54375) (end 224.5 29.5875) (width 1) (layer F.Cu) (net 1))
@@
   (segment (start 199.5 29.5) (end 199.5 37.42) (width 3) (layer F.Cu) (net 2))
   (segment (start 205.575 29.5) (end 199.5 29.5) (width 1) (layer F.Cu) (net 2))
-  (via (at 225.25 69) (size 1.4) (drill 0.7) (layers F.Cu B.Cu) (net 2))
-  (segment (start 205.75 35.75) (end 199.5 29.5) (width 2) (layer B.Cu) (net 2))
-  (segment (start 205.75 42.762602) (end 205.75 35.75) (width 2) (layer B.Cu) (net 2))
-  (segment (start 225.25 69) (end 224 69) (width 2) (layer B.Cu) (net 2))
-  (segment (start 219.5 64.5) (end 219.5 56.512602) (width 2) (layer B.Cu) (net 2))
-  (segment (start 219.5 56.512602) (end 205.75 42.762602) (width 2) (layer B.Cu) (net 2))
-  (segment (start 224 69) (end 219.5 64.5) (width 2) (layer B.Cu) (net 2))
+  (segment (start 219.5 64.5) (end 219.5 56.512602) (width 2) (layer B.Cu) (net 2) (status 1000000))
+  (segment (start 205.75 35.75) (end 199.5 29.5) (width 2) (layer B.Cu) (net 2) (status 1000000))
+  (segment (start 224 69) (end 219.5 64.5) (width 2) (layer B.Cu) (net 2) (status 1000000))
+  (segment (start 219.5 56.512602) (end 205.75 42.762602) (width 2) (layer B.Cu) (net 2) (status 1000000))
+  (via (at 225.25 69) (size 1.4) (drill 0.7) (layers F.Cu B.Cu) (net 2) (status 1000000))
+  (segment (start 205.75 42.762602) (end 205.75 35.75) (width 2) (layer B.Cu) (net 2) (status 1000000))
+  (segment (start 225.25 69) (end 224 69) (width 2) (layer B.Cu) (net 2) (status 1000000))
   (segment (start 227.2775 69) (end 227.2775 69) (width 0.6) (layer F.Cu) (net 3))
   (segment (start 227.2775 69) (end 229.3 69) (width 0.6) (layer F.Cu) (net 3))
